File: design/pro_030_mini/kicad/CPU.sch (KiCad schematic (older format))
At the start: 23 parts, among them IC1 MC68030RC_PGA

Commit message: Update footprints for pro 030 mini
Parts:
- added X1: CXO_DIP8, Oscillator:Oscillator_DIP-8, symbol Oscillator:CXO_DIP8
Connections:
- net GND: now also X1.1 (EN), X1.4 (GND)
- net VCC: now also IC1.F13 (MMUDIS), IC1.G1 (STERM), IC1.H12 (CDIS), IC1.J1 (CBACK), X1.8 (Vcc)
- net BR: now reaches IC1.A1 (BR)
- net A17: now reaches IC1.A10 (A17)
- net A15: now reaches IC1.A11 (A15)
- net A13: now reaches IC1.A12 (A13)
- net A10: now reaches IC1.A13 (A10)
- net A0: now reaches IC1.A2 (A0)
- net A30: now reaches IC1.A3 (A30)
- net A28: now reaches IC1.A4 (A28)
- net A26: now reaches IC1.A5 (A26)
- net A24: now reaches IC1.A6 (A24)
- net A23: now reaches IC1.A7 (A23)
- net A21: now reaches IC1.A8 (A21)
- net A19: now reaches IC1.A9 (A19)
- net RMC: now reaches IC1.B1 (RMC)
- net A14: now reaches IC1.B10 (A14)
- net A12: now reaches IC1.B11 (A12)
- net A8: now reaches IC1.B12 (A8)
- net A7: now reaches IC1.B13 (A7)
- net BG: now reaches IC1.B2 (BG)
- net A31: now reaches IC1.B3 (A31)
- net A29: now reaches IC1.B4 (A29)
- net A27: now reaches IC1.B5 (A27)
- net A25: now reaches IC1.B6 (A25)
- net A22: now reaches IC1.B7 (A22)
- net A20: now reaches IC1.B8 (A20)
- net A16: now reaches IC1.B9 (A16)
- net FC1: now reaches IC1.C1 (FC1)
- net A11: now reaches IC1.C10 (A11)
- net A9: now reaches IC1.C11 (A9)
- net A5: now reaches IC1.C12 (A5)
- net A4: now reaches IC1.C13 (A4)
- net BGACK: now reaches IC1.C3 (BGACK)
- net A1: now reaches IC1.C4 (A1)
- net A18: now reaches IC1.C8 (A18)
- net FC2: now reaches IC1.D1 (FC2)
- net A6: now reaches IC1.D11 (A6)
- net A3: now reaches IC1.D12 (A3)
- net A2: now reaches IC1.D13 (A2)
- net FC0: now reaches IC1.D2 (FC0)
- net CLK: now reaches IC1.E1 (CLKIN)
- net CLK: now also X1.5 (OUT)
- net IPEND: now reaches IC1.E13 (IPEND)
- net AVEC: now reaches IC1.E2 (AVEC)
- net DSACK0: now reaches IC1.F1 (DSACK0)
- net RESET: now reaches IC1.F12 (RESET)
- net IPL2: now reaches IC1.G12 (IPL2)
- net IPL1: now reaches IC1.G13 (IPL1)
- net DSACK1: now reaches IC1.G2 (DSACK1)
- net BERR: now reaches IC1.H1 (BERR)
- net IPL0: now reaches IC1.H13 (IPL0)
- net HALT: now reaches IC1.H2 (HLT)
- net AS: now reaches IC1.J2 (AS)
- net D5: now reaches IC1.K11 (D5)
- net D1: now reaches IC1.K12 (D1)
- net D0: now reaches IC1.K13 (D0)
- net DS: now reaches IC1.K2 (DS)
- net SIZ1: now reaches IC1.K3 (SIZ1)
- net CIIN: now reaches IC1.L1 (CIIN)
- net D10: now reaches IC1.L10 (D10)
- net D7: now reaches IC1.L11 (D7)
- net D4: now reaches IC1.L12 (D4)
- net D2: now reaches IC1.L13 (D2)
- net SIZ0: now reaches IC1.L2 (SIZ0)
- net RW: now reaches IC1.L3 (R_W)
- net D30: now reaches IC1.L4 (D30)
- net DBEN: now reaches IC1.M1 (DBEN)
- net D12: now reaches IC1.M10 (D12)
- net D9: now reaches IC1.M11 (D9)
- net D6: now reaches IC1.M12 (D6)
- net D3: now reaches IC1.M13 (D3)
- net D29: now reaches IC1.M3 (D29)
- net D27: now reaches IC1.M4 (D27)
- net D24: now reaches IC1.M5 (D24)
- net D22: now reaches IC1.M6 (D22)
- net D20: now reaches IC1.M7 (D20)
- net D17: now reaches IC1.M8 (D17)
- net D14: now reaches IC1.M9 (D14)
- net D31: now reaches IC1.N1 (D31)
- net D15: now reaches IC1.N10 (D15)
- net D13: now reaches IC1.N11 (D13)
- net D11: now reaches IC1.N12 (D11)
- net D8: now reaches IC1.N13 (D8)
- net D28: now reaches IC1.N2 (D28)
- net D26: now reaches IC1.N3 (D26)
- net D25: now reaches IC1.N4 (D25)
- net D23: now reaches IC1.N5 (D23)
- net D21: now reaches IC1.N6 (D21)
- net D19: now reaches IC1.N7 (D19)
- net D18: now reaches IC1.N8 (D18)
- net D16: now reaches IC1.N9 (D16)
- no-connect marks 0 -> 6
Other:
- note added: "TODO needs correct footprint etc…"
