File: design/pro_030_proto/kicad/GLUE.sch (KiCad schematic (older format))
At the start: 19 parts, among them IC4 74174N, IC5 74HCT93, IC6 74LS08, IC7 74HCT93, IC8 74HCT174, IC9 74LS01N, X2 8MHz

Commit message: Further layout
Parts:
- renumbered C13 to C12, C14 to C13, IC4 to IC3, IC5 to IC4, IC6 to IC5, IC7 to IC6, IC8 to IC7, IC9 to IC8
Changed lines of the file:
@@
 AR Path="/5E53B810/60F55293" Ref="IC?"  Part="1"
 AR Path="/5E53B952/60F55293" Ref="IC?"  Part="1"
-AR Path="/60FBFA5C/60F55293" Ref="IC4"  Part="1"
-F 0 "IC4" H 2950 2075 59  0000 L BNN
+AR Path="/60FBFA5C/60F55293" Ref="IC3"  Part="1"
+F 0 "IC3" H 2950 2075 59  0000 L BNN
 F 1 "74174N" H 2950 950 59  0000 L BNN
 F 2 "Package_DIP:DIP-16_W7.62mm_Socket_LongPads" H 3250 1550 50  0001 C CNN
@@
 AR Path="/5E53B952/60F552BD" Ref="IC?"  Part="4"
 AR Path="/5E53BC83/60F552BD" Ref="IC?"  Part="4"
-AR Path="/60FBFA5C/60F552BD" Ref="IC9"  Part="4"
-F 0 "IC9" H 10050 1825 59  0000 L BNN
+AR Path="/60FBFA5C/60F552BD" Ref="IC8"  Part="4"
+F 0 "IC8" H 10050 1825 59  0000 L BNN
 F 1 "74LS01N" H 10050 1500 59  0001 L BNN
 F 2 "Package_DIP:DIP-14_W7.62mm_Socket_LongPads" H 9950 1700 50  0001 C CNN
@@
 	8550 2000 8550 2200
 $Comp
-L power:GND #PWR028
+L power:GND #PWR027
 U 1 1 60F552C7
 P 8550 2200
-F 0 "#PWR028" H 8550 1950 50  0001 C CNN
+F 0 "#PWR027" H 8550 1950 50  0001 C CNN
 F 1 "GND" H 8555 2027 50  0000 C CNN
 F 2 "" H 8550 2200 50  0001 C CNN
@@
 $EndComp
 $Comp
-L power:VCC #PWR027
+L power:VCC #PWR026
 U 1 1 60F552CD
 P 8550 750
-F 0 "#PWR027" H 8550 600 50  0001 C CNN
+F 0 "#PWR026" H 8550 600 50  0001 C CNN
 F 1 "VCC" H 8567 923 50  0000 C CNN
 F 2 "" H 8550 750 50  0001 C CNN
@@
 AS
 $Comp
-L 74xx:74LS93 IC7
+L 74xx:74LS93 IC6
 U 1 1 60F552E6
 P 8550 1500
-F 0 "IC7" H 8350 1900 50  0000 C CNN
+F 0 "IC6" H 8350 1900 50  0000 C CNN
 F 1 "74HCT93" H 8750 1900 50  0000 C CNN
 F 2 "Package_DIP:DIP-14_W7.62mm_Socket_LongPads" H 8550 1500 50  0001 C CNN
@@
 $EndComp
 $Comp
-L 74xx:74LS08 IC6
+L 74xx:74LS08 IC5
 U 1 1 60FBB5A0
 P 7350 1700
-F 0 "IC6" H 7350 2025 50  0000 C CNN
+F 0 "IC5" H 7350 2025 50  0000 C CNN
 F 1 "74LS08" H 7350 1934 50  0000 C CNN
 F 2 "Package_DIP:DIP-14_W7.62mm_LongPads" H 7350 1700 50  0001 C CNN
@@
 	8550 750  8550 1000
 $Comp
-L 74xx:74LS174 IC8
+L 74xx:74LS174 IC7
 U 1 1 60FDF4F7
 P 8600 4150
-F 0 "IC8" H 8600 5031 50  0000 C CNN
+F 0 "IC7" H 8600 5031 50  0000 C CNN
 F 1 "74HCT174" H 8600 4940 50  0000 C CNN
 F 2 "Package_DIP:DIP-16_W7.62mm_Socket_LongPads" H 8600 4150 50  0001 C CNN
@@
 AR Path="/6100331A" Ref="C?"  Part="1"
 AR Path="/5E53B952/6100331A" Ref="C?"  Part="1"
-AR Path="/60FBFA5C/6100331A" Ref="C14"  Part="1"
-F 0 "C14" H 8110 4965 59  0000 L BNN
+AR Path="/60FBFA5C/6100331A" Ref="C13"  Part="1"
+F 0 "C13" H 8110 4965 59  0000 L BNN
 F 1 "100nF" H 8110 4765 59  0000 L BNN
 F 2 "Capacitor_THT:C_Rect_L4.0mm_W2.5mm_P2.50mm" H 8050 4950 50  0001 C CNN
@@
 	8600 5150 8600 4950
 $Comp
-L power:GND #PWR029
+L power:GND #PWR028
 U 1 1 61012297
 P 8600 5150
-F 0 "#PWR029" H 8600 4900 50  0001 C CNN
+F 0 "#PWR028" H 8600 4900 50  0001 C CNN
 F 1 "GND" H 8605 4977 50  0000 C CNN
 F 2 "" H 8600 5150 50  0001 C CNN
@@
 Connection ~ 8600 5150
 $Comp
-L power:VCC #PWR026
+L power:VCC #PWR025
 U 1 1 610129A0
 P 8050 3450
-F 0 "#PWR026" H 8050 3300 50  0001 C CNN
+F 0 "#PWR025" H 8050 3300 50  0001 C CNN
 F 1 "VCC" H 8067 3623 50  0000 C CNN
 F 2 "" H 8050 3450 50  0001 C CNN
@@
 AR Path="/6109A096" Ref="C?"  Part="1"
 AR Path="/5E53B952/6109A096" Ref="C?"  Part="1"
-AR Path="/60FBFA5C/6109A096" Ref="C13"  Part="1"
-F 0 "C13" H 4310 5565 59  0000 L BNN
+AR Path="/60FBFA5C/6109A096" Ref="C12"  Part="1"
+F 0 "C12" H 4310 5565 59  0000 L BNN
 F 1 "100nF" H 4310 5365 59  0000 L BNN
 F 2 "Capacitor_THT:C_Rect_L4.0mm_W2.5mm_P2.50mm" H 4250 5550 50  0001 C CNN
@@
 P 1800 5500
 AR Path="/60EC67C5/61242933" Ref="#PWR?"  Part="1"
-AR Path="/60FBFA5C/61242933" Ref="#PWR023"  Part="1"
-F 0 "#PWR023" H 1800 5250 50  0001 C CNN
+AR Path="/60FBFA5C/61242933" Ref="#PWR019"  Part="1"
+F 0 "#PWR019" H 1800 5250 50  0001 C CNN
 F 1 "GND" H 1805 5327 50  0000 C CNN
 F 2 "" H 1800 5500 50  0001 C CNN
@@
 P 1800 4350
 AR Path="/60EC67C5/6124292D" Ref="#PWR?"  Part="1"
-AR Path="/60FBFA5C/6124292D" Ref="#PWR022"  Part="1"
-F 0 "#PWR022" H 1800 4200 50  0001 C CNN
+AR Path="/60FBFA5C/6124292D" Ref="#PWR018"  Part="1"
+F 0 "#PWR018" H 1800 4200 50  0001 C CNN
 F 1 "VCC" H 1817 4523 50  0000 C CNN
 F 2 "" H 1800 4350 50  0001 C CNN
@@
 	3300 5800 2550 5800
 $Comp
-L power:GND #PWR025
+L power:GND #PWR023
 U 1 1 61089066
 P 3300 5950
-F 0 "#PWR025" H 3300 5700 50  0001 C CNN
+F 0 "#PWR023" H 3300 5700 50  0001 C CNN
 F 1 "GND" H 3305 5777 50  0000 C CNN
 F 2 "" H 3300 5950 50  0001 C CNN
@@
 $EndComp
 $Comp
-L power:VCC #PWR024
+L power:VCC #PWR022
 U 1 1 6108898F
 P 3300 4450
-F 0 "#PWR024" H 3300 4300 50  0001 C CNN
+F 0 "#PWR022" H 3300 4300 50  0001 C CNN
 F 1 "VCC" H 3317 4623 50  0000 C CNN
 F 2 "" H 3300 4450 50  0001 C CNN
@@
 	3800 4900 4050 4900
 $Comp
-L 74xx:74LS93 IC5
+L 74xx:74LS93 IC4
 U 1 1 6107269E
 P 3300 5100
-F 0 "IC5" H 3100 5500 50  0000 C CNN
+F 0 "IC4" H 3100 5500 50  0000 C CNN
 F 1 "74HCT93" H 3500 5500 50  0000 C CNN
 F 2 "Package_DIP:DIP-14_W7.62mm_Socket_LongPads" H 3300 5100 50  0001 C CNN
@@
 $EndComp
 $Comp
-L 74xx:74LS08 IC6
+L 74xx:74LS08 IC5
 U 2 1 614E4FA8
 P 5800 5750
-F 0 "IC6" H 5800 6075 50  0000 C CNN
+F 0 "IC5" H 5800 6075 50  0000 C CNN
 F 1 "74LS08" H 5800 5984 50  0000 C CNN
 F 2 "Package_DIP:DIP-14_W7.62mm_LongPads" H 5800 5750 50  0001 C CNN
@@
 $EndComp
 $Comp
-L 74xx:74LS08 IC6
+L 74xx:74LS08 IC5
 U 3 1 614EBD83
 P 5800 6350
-F 0 "IC6" H 5800 6675 50  0000 C CNN
+F 0 "IC5" H 5800 6675 50  0000 C CNN
 F 1 "74LS08" H 5800 6584 50  0000 C CNN
 F 2 "Package_DIP:DIP-14_W7.62mm_LongPads" H 5800 6350 50  0001 C CNN
@@
 $EndComp
 $Comp
-L 74xx:74LS08 IC6
+L 74xx:74LS08 IC5
 U 4 1 614F28BB
 P 5800 6950
-F 0 "IC6" H 5800 7275 50  0000 C CNN
+F 0 "IC5" H 5800 7275 50  0000 C CNN
 F 1 "74LS08" H 5800 7184 50  0000 C CNN
 F 2 "Package_DIP:DIP-14_W7.62mm_LongPads" H 5800 6950 50  0001 C CNN
@@
 $EndComp
 $Comp
-L power:GND #PWR0101
+L power:GND #PWR024
 U 1 1 614F7B04
 P 5250 7350
-F 0 "#PWR0101" H 5250 7100 50  0001 C CNN
+F 0 "#PWR024" H 5250 7100 50  0001 C CNN
 F 1 "GND" H 5255 7177 50  0000 C CNN
 F 2 "" H 5250 7350 50  0001 C CNN

Commit message: Add IO and XVID glue etc.
* Add IO Select glue
* Add Xosera glue
* Add new glues to schematic
* Clean up libs
* Reannotate (again)
Parts:
- renumbered IC4 to IC10, IC5 to IC11, IC6 to IC12, IC7 to IC13, IC8 to IC14, IC3 to IC9
Changed lines of the file:
@@
 AR Path="/5E53B810/60F55293" Ref="IC?"  Part="1"
 AR Path="/5E53B952/60F55293" Ref="IC?"  Part="1"
-AR Path="/60FBFA5C/60F55293" Ref="IC3"  Part="1"
-F 0 "IC3" H 2950 2075 59  0000 L BNN
+AR Path="/60FBFA5C/60F55293" Ref="IC9"  Part="1"
+F 0 "IC9" H 2950 2075 59  0000 L BNN
 F 1 "74174N" H 2950 950 59  0000 L BNN
 F 2 "Package_DIP:DIP-16_W7.62mm_Socket_LongPads" H 3250 1550 50  0001 C CNN
@@
 AR Path="/5E53B952/60F552BD" Ref="IC?"  Part="4"
 AR Path="/5E53BC83/60F552BD" Ref="IC?"  Part="4"
-AR Path="/60FBFA5C/60F552BD" Ref="IC8"  Part="4"
-F 0 "IC8" H 10050 1825 59  0000 L BNN
+AR Path="/60FBFA5C/60F552BD" Ref="IC14"  Part="4"
+F 0 "IC14" H 10050 1825 59  0000 L BNN
 F 1 "74LS01N" H 10050 1500 59  0001 L BNN
 F 2 "Package_DIP:DIP-14_W7.62mm_Socket_LongPads" H 9950 1700 50  0001 C CNN
@@
 AS
 $Comp
-L 74xx:74LS93 IC6
+L 74xx:74LS93 IC12
 U 1 1 60F552E6
 P 8550 1500
-F 0 "IC6" H 8350 1900 50  0000 C CNN
+F 0 "IC12" H 8350 1900 50  0000 C CNN
 F 1 "74HCT93" H 8750 1900 50  0000 C CNN
 F 2 "Package_DIP:DIP-14_W7.62mm_Socket_LongPads" H 8550 1500 50  0001 C CNN
@@
 $EndComp
 $Comp
-L 74xx:74LS08 IC5
+L 74xx:74LS08 IC11
 U 1 1 60FBB5A0
 P 7350 1700
-F 0 "IC5" H 7350 2025 50  0000 C CNN
+F 0 "IC11" H 7350 2025 50  0000 C CNN
 F 1 "74LS08" H 7350 1934 50  0000 C CNN
 F 2 "Package_DIP:DIP-14_W7.62mm_LongPads" H 7350 1700 50  0001 C CNN
@@
 	8550 750  8550 1000
 $Comp
-L 74xx:74LS174 IC7
+L 74xx:74LS174 IC13
 U 1 1 60FDF4F7
 P 8600 4150
-F 0 "IC7" H 8600 5031 50  0000 C CNN
+F 0 "IC13" H 8600 5031 50  0000 C CNN
 F 1 "74HCT174" H 8600 4940 50  0000 C CNN
 F 2 "Package_DIP:DIP-16_W7.62mm_Socket_LongPads" H 8600 4150 50  0001 C CNN
@@
 	3800 4900 4050 4900
 $Comp
-L 74xx:74LS93 IC4
+L 74xx:74LS93 IC10
 U 1 1 6107269E
 P 3300 5100
-F 0 "IC4" H 3100 5500 50  0000 C CNN
+F 0 "IC10" H 3100 5500 50  0000 C CNN
 F 1 "74HCT93" H 3500 5500 50  0000 C CNN
 F 2 "Package_DIP:DIP-14_W7.62mm_Socket_LongPads" H 3300 5100 50  0001 C CNN
@@
 $EndComp
 $Comp
-L 74xx:74LS08 IC5
+L 74xx:74LS08 IC11
 U 2 1 614E4FA8
 P 5800 5750
-F 0 "IC5" H 5800 6075 50  0000 C CNN
+F 0 "IC11" H 5800 6075 50  0000 C CNN
 F 1 "74LS08" H 5800 5984 50  0000 C CNN
 F 2 "Package_DIP:DIP-14_W7.62mm_LongPads" H 5800 5750 50  0001 C CNN
@@
 $EndComp
 $Comp
-L 74xx:74LS08 IC5
+L 74xx:74LS08 IC11
 U 3 1 614EBD83
 P 5800 6350
-F 0 "IC5" H 5800 6675 50  0000 C CNN
+F 0 "IC11" H 5800 6675 50  0000 C CNN
 F 1 "74LS08" H 5800 6584 50  0000 C CNN
 F 2 "Package_DIP:DIP-14_W7.62mm_LongPads" H 5800 6350 50  0001 C CNN
@@
 $EndComp
 $Comp
-L 74xx:74LS08 IC5
+L 74xx:74LS08 IC11
 U 4 1 614F28BB
 P 5800 6950
-F 0 "IC5" H 5800 7275 50  0000 C CNN
+F 0 "IC11" H 5800 7275 50  0000 C CNN
 F 1 "74LS08" H 5800 7184 50  0000 C CNN
 F 2 "Package_DIP:DIP-14_W7.62mm_LongPads" H 5800 6950 50  0001 C CNN
