File: design/pro_030_proto/kicad/LEVELSHIFT.sch (KiCad schematic (older format))
At the start: 20 parts, among them IC21 74HCT245, IC22 74HCT245, IC23 74HCT245, IC24 74HCT245

Commit message: Further layout
Parts:
- added C54, C55, C56, C57, C58, C59, C60, C61: 100nF, rosco_m68k:C2.5-3, symbol Device:C
- added IC24, IC25, IC26, IC27: 74HCT245, Package_DIP:DIP-20_W7.62mm_Socket_LongPads, symbol 74xx:74LS245
- added R58, R59, R60, R61, R62, R63, R64, R65, R66, R67, R68, R69, R70, R71, R72, R73: R, rosco_m68k:R-0207_10, symbol Device:R
- renumbered IC21 to IC20, IC22 to IC21, IC23 to IC22, IC24 to IC23, R44 to R42, R45 to R43, R46 to R44, R47 to R45, R48 to R46, R49 to R47, R50 to R48, R51 to R49, R52 to R50, R53 to R51, R54 to R52, R55 to R53, R56 to R54, R57 to R55, R58 to R56, R59 to R57
Connections:
- net 3V3: now also C54.1, C55.1, C56.1, C57.1, IC24.20 (VCC), IC26.20 (VCC)
- net 5V: now also C58.1, C59.1, C60.1, C61.1, IC25.20 (VCC), IC27.20 (VCC)
- net GND: now also C54.2, C55.2, C56.2, C57.2, C58.2, C59.2, C60.2, C61.2, IC24.1 (A->B), IC24.10 (GND), IC25.1 (A->B), IC25.10 (GND), IC26.1 (A->B), IC26.10 (GND), IC27.1 (A->B), IC27.10 (GND)
- net LV_R: now also IC25.19 (CE), IC27.19 (CE)
- net LV_W: now also IC24.19 (CE), IC26.19 (CE)
- new net: IC24.11 (B7), R65.2
- new net: IC24.12 (B6), R64.2
- new net: IC24.13 (B5), R63.2
- new net: IC24.14 (B4), R62.2
- new net: IC24.15 (B3), R61.2
- new net: IC24.16 (B2), R60.2
- new net: IC24.17 (B1), R59.2
- new net: IC24.18 (B0), R58.2
- new net: IC26.11 (B7), R73.2
- new net: IC26.12 (B6), R72.2
- new net: IC26.13 (B5), R71.2
- new net: IC26.14 (B4), R70.2
- new net: IC26.15 (B3), R69.2
- new net: IC26.16 (B2), R68.2
- new net: IC26.17 (B1), R67.2
- new net: IC26.18 (B0), R66.2
- new net 3V3_D16: IC24.9 (A7), IC25.11 (B7)
- new net 3V3_D17: IC24.8 (A6), IC25.12 (B6)
- new net 3V3_D18: IC24.7 (A5), IC25.13 (B5)
- new net 3V3_D19: IC24.6 (A4), IC25.14 (B4)
- new net 3V3_D20: IC24.5 (A3), IC25.15 (B3)
- new net 3V3_D21: IC24.4 (A2), IC25.16 (B2)
- new net 3V3_D22: IC24.3 (A1), IC25.17 (B1)
- new net 3V3_D23: IC24.2 (A0), IC25.18 (B0)
- new net 3V3_D24: IC26.9 (A7), IC27.11 (B7)
- new net 3V3_D25: IC26.8 (A6), IC27.12 (B6)
- new net 3V3_D26: IC26.7 (A5), IC27.13 (B5)
- new net 3V3_D27: IC26.6 (A4), IC27.14 (B4)
- new net 3V3_D28: IC26.5 (A3), IC27.15 (B3)
- new net 3V3_D29: IC26.4 (A2), IC27.16 (B2)
- new net 3V3_D30: IC26.3 (A1), IC27.17 (B1)
- new net 3V3_D31: IC26.2 (A0), IC27.18 (B0)
- new net 68_D16: IC25.9 (A7), R65.1
- new net 68_D17: IC25.8 (A6), R64.1
- new net 68_D18: IC25.7 (A5), R63.1
- new net 68_D19: IC25.6 (A4), R62.1
- new net 68_D20: IC25.5 (A3), R61.1
- new net 68_D21: IC25.4 (A2), R60.1
- new net 68_D22: IC25.3 (A1), R59.1
- new net 68_D23: IC25.2 (A0), R58.1
- new net 68_D24: IC27.9 (A7), R73.1
- new net 68_D25: IC27.8 (A6), R72.1
- new net 68_D26: IC27.7 (A5), R71.1
- new net 68_D27: IC27.6 (A4), R70.1
- new net 68_D28: IC27.5 (A3), R69.1
- new net 68_D29: IC27.4 (A2), R68.1
- new net 68_D30: IC27.3 (A1), R67.1
- new net 68_D31: IC27.2 (A0), R66.1
Other:
- moved on the sheet: IC20, IC21, IC22, IC23, R42, R43, R44, R45, R46, R47, R48, R49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

Commit message: Add IO and XVID glue etc.
* Add IO Select glue
* Add Xosera glue
* Add new glues to schematic
* Clean up libs
* Reannotate (again)
Parts:
- renumbered C54 to C56, C55 to C57, C56 to C58, C57 to C59, C58 to C60, C59 to C61, C60 to C62, C61 to C63
Changed lines of the file:
@@
 P 1250 1000
 AR Path="/61161E57/6154492D" Ref="C?"  Part="1"
-AR Path="/6116F31D/6154492D" Ref="C54"  Part="1"
-F 0 "C54" H 1365 1046 50  0000 L CNN
+AR Path="/6116F31D/6154492D" Ref="C56"  Part="1"
+F 0 "C56" H 1365 1046 50  0000 L CNN
 F 1 "100nF" H 1365 955 50  0000 L CNN
 F 2 "rosco_m68k:C2.5-3" H 1288 850 50  0001 C CNN
@@
 P 1750 1000
 AR Path="/61161E57/6154763A" Ref="C?"  Part="1"
-AR Path="/6116F31D/6154763A" Ref="C55"  Part="1"
-F 0 "C55" H 1865 1046 50  0000 L CNN
+AR Path="/6116F31D/6154763A" Ref="C57"  Part="1"
+F 0 "C57" H 1865 1046 50  0000 L CNN
 F 1 "100nF" H 1865 955 50  0000 L CNN
 F 2 "rosco_m68k:C2.5-3" H 1788 850 50  0001 C CNN
@@
 P 2250 1000
 AR Path="/61161E57/6154A27E" Ref="C?"  Part="1"
-AR Path="/6116F31D/6154A27E" Ref="C56"  Part="1"
-F 0 "C56" H 2365 1046 50  0000 L CNN
+AR Path="/6116F31D/6154A27E" Ref="C58"  Part="1"
+F 0 "C58" H 2365 1046 50  0000 L CNN
 F 1 "100nF" H 2365 955 50  0000 L CNN
 F 2 "rosco_m68k:C2.5-3" H 2288 850 50  0001 C CNN
@@
 P 2800 1000
 AR Path="/61161E57/6154D384" Ref="C?"  Part="1"
-AR Path="/6116F31D/6154D384" Ref="C57"  Part="1"
-F 0 "C57" H 2915 1046 50  0000 L CNN
+AR Path="/6116F31D/6154D384" Ref="C59"  Part="1"
+F 0 "C59" H 2915 1046 50  0000 L CNN
 F 1 "100nF" H 2915 955 50  0000 L CNN
 F 2 "rosco_m68k:C2.5-3" H 2838 850 50  0001 C CNN
@@
 P 8750 1050
 AR Path="/61161E57/61551048" Ref="C?"  Part="1"
-AR Path="/6116F31D/61551048" Ref="C58"  Part="1"
-F 0 "C58" H 8865 1096 50  0000 L CNN
+AR Path="/6116F31D/61551048" Ref="C60"  Part="1"
+F 0 "C60" H 8865 1096 50  0000 L CNN
 F 1 "100nF" H 8865 1005 50  0000 L CNN
 F 2 "rosco_m68k:C2.5-3" H 8788 900 50  0001 C CNN
@@
 P 9250 1050
 AR Path="/61161E57/6155104E" Ref="C?"  Part="1"
-AR Path="/6116F31D/6155104E" Ref="C59"  Part="1"
-F 0 "C59" H 9365 1096 50  0000 L CNN
+AR Path="/6116F31D/6155104E" Ref="C61"  Part="1"
+F 0 "C61" H 9365 1096 50  0000 L CNN
 F 1 "100nF" H 9365 1005 50  0000 L CNN
 F 2 "rosco_m68k:C2.5-3" H 9288 900 50  0001 C CNN
@@
 P 9750 1050
 AR Path="/61161E57/61551054" Ref="C?"  Part="1"
-AR Path="/6116F31D/61551054" Ref="C60"  Part="1"
-F 0 "C60" H 9865 1096 50  0000 L CNN
+AR Path="/6116F31D/61551054" Ref="C62"  Part="1"
+F 0 "C62" H 9865 1096 50  0000 L CNN
 F 1 "100nF" H 9865 1005 50  0000 L CNN
 F 2 "rosco_m68k:C2.5-3" H 9788 900 50  0001 C CNN
@@
 P 10300 1050
 AR Path="/61161E57/6155105A" Ref="C?"  Part="1"
-AR Path="/6116F31D/6155105A" Ref="C61"  Part="1"
-F 0 "C61" H 10415 1096 50  0000 L CNN
+AR Path="/6116F31D/6155105A" Ref="C63"  Part="1"
+F 0 "C63" H 10415 1096 50  0000 L CNN
 F 1 "100nF" H 10415 1005 50  0000 L CNN
 F 2 "rosco_m68k:C2.5-3" H 10338 900 50  0001 C CNN

Commit message: First cut placement
Parts:
- C56, C57, C58, C59, C60, C61, C62, C63: footprint rosco_m68k:C2.5-3 -> Capacitor_THT:C_Rect_L4.0mm_W2.5mm_P2.50mm
Changed lines of the file:
@@
 F 0 "C56" H 1365 1046 50  0000 L CNN
 F 1 "100nF" H 1365 955 50  0000 L CNN
-F 2 "rosco_m68k:C2.5-3" H 1288 850 50  0001 C CNN
+F 2 "Capacitor_THT:C_Rect_L4.0mm_W2.5mm_P2.50mm" H 1288 850 50  0001 C CNN
 F 3 "~" H 1250 1000 50  0001 C CNN
 	1    1250 1000
@@
 F 0 "C57" H 1865 1046 50  0000 L CNN
 F 1 "100nF" H 1865 955 50  0000 L CNN
-F 2 "rosco_m68k:C2.5-3" H 1788 850 50  0001 C CNN
+F 2 "Capacitor_THT:C_Rect_L4.0mm_W2.5mm_P2.50mm" H 1788 850 50  0001 C CNN
 F 3 "~" H 1750 1000 50  0001 C CNN
 	1    1750 1000
@@
 F 0 "C58" H 2365 1046 50  0000 L CNN
 F 1 "100nF" H 2365 955 50  0000 L CNN
-F 2 "rosco_m68k:C2.5-3" H 2288 850 50  0001 C CNN
+F 2 "Capacitor_THT:C_Rect_L4.0mm_W2.5mm_P2.50mm" H 2288 850 50  0001 C CNN
 F 3 "~" H 2250 1000 50  0001 C CNN
 	1    2250 1000
@@
 F 0 "C59" H 2915 1046 50  0000 L CNN
 F 1 "100nF" H 2915 955 50  0000 L CNN
-F 2 "rosco_m68k:C2.5-3" H 2838 850 50  0001 C CNN
+F 2 "Capacitor_THT:C_Rect_L4.0mm_W2.5mm_P2.50mm" H 2838 850 50  0001 C CNN
 F 3 "~" H 2800 1000 50  0001 C CNN
 	1    2800 1000
@@
 F 0 "C60" H 8865 1096 50  0000 L CNN
 F 1 "100nF" H 8865 1005 50  0000 L CNN
-F 2 "rosco_m68k:C2.5-3" H 8788 900 50  0001 C CNN
+F 2 "Capacitor_THT:C_Rect_L4.0mm_W2.5mm_P2.50mm" H 8788 900 50  0001 C CNN
 F 3 "~" H 8750 1050 50  0001 C CNN
 	1    8750 1050
@@
 F 0 "C61" H 9365 1096 50  0000 L CNN
 F 1 "100nF" H 9365 1005 50  0000 L CNN
-F 2 "rosco_m68k:C2.5-3" H 9288 900 50  0001 C CNN
+F 2 "Capacitor_THT:C_Rect_L4.0mm_W2.5mm_P2.50mm" H 9288 900 50  0001 C CNN
 F 3 "~" H 9250 1050 50  0001 C CNN
 	1    9250 1050
@@
 F 0 "C62" H 9865 1096 50  0000 L CNN
 F 1 "100nF" H 9865 1005 50  0000 L CNN
-F 2 "rosco_m68k:C2.5-3" H 9788 900 50  0001 C CNN
+F 2 "Capacitor_THT:C_Rect_L4.0mm_W2.5mm_P2.50mm" H 9788 900 50  0001 C CNN
 F 3 "~" H 9750 1050 50  0001 C CNN
 	1    9750 1050
@@
 F 0 "C63" H 10415 1096 50  0000 L CNN
 F 1 "100nF" H 10415 1005 50  0000 L CNN
-F 2 "rosco_m68k:C2.5-3" H 10338 900 50  0001 C CNN
+F 2 "Capacitor_THT:C_Rect_L4.0mm_W2.5mm_P2.50mm" H 10338 900 50  0001 C CNN
 F 3 "~" H 10300 1050 50  0001 C CNN
 	1    10300 1050
