File: design/pro_030_proto/kicad/RESET.sch (KiCad schematic (older format))
At the start: 15 parts

Commit message: Largeish changeset:
* Added (first-cut) glue for DTACK generation
* Fix mem selects to use new DTACK generation
* Add missing footprints for Kicad
* Add POWER and TESTPOINTS schematics
* Update footprints across the board to allow error-free PCB import
* Pull all components (so far) into PCB
* Fix MC68030RC footprint (missing pads)
Parts:
- C10: renamed from C?; footprint rosco_m68k:E2,5-5 -> rosco_m68k:C-Electolytic-2,5-5
- R26, R27, R28, R29, R30, R31: renamed from R?; footprint rosco_m68k:0207_10 -> rosco_m68k:R-0207_10
- gave numbers to parts that had none: 6
Changed lines of the file:
@@
 $Descr A4 11693 8268
 encoding utf-8
-Sheet 8 8
-Title ""
-Date ""
-Rev ""
-Comp ""
-Comment1 ""
-Comment2 ""
-Comment3 ""
+Sheet 8 10
+Title "rosco_m68k Pro (030) Prototype"
+Date "2021-07-24"
+Rev "0"
+Comp "The Really Old-School Company Limited"
+Comment1 "Copyright ©2021 The Really Old-School Company Limited"
+Comment2 "Open Source Hardware (CERN OHL)"
+Comment3 "Prototype Hardware! Not suitable for general use!"
 Comment4 ""
 $EndDescr
@@
 AR Path="/5E53B952/6104F00C" Ref="IC?"  Part="1"
 AR Path="/60FBFA5C/6104F00C" Ref="IC?"  Part="1"
-F 0 "IC?" H 3850 4130 59  0000 L BNN
+AR Path="/61043B8D/6104F00C" Ref="IC10"  Part="1"
+F 0 "IC10" H 3850 4130 59  0000 L BNN
 F 1 "555N" H 3850 3195 59  0000 L BNN
 F 2 "Package_DIP:DIP-8_W7.62mm_LongPads" H 4150 3700 50  0001 C CNN
@@
 AR Path="/5E53B952/6104F012" Ref="IC?"  Part="1"
 AR Path="/60FBFA5C/6104F012" Ref="IC?"  Part="1"
-F 0 "IC?" H 5900 4925 59  0000 L BNN
+AR Path="/61043B8D/6104F012" Ref="IC9"  Part="1"
+F 0 "IC9" H 5900 4925 59  0000 L BNN
 F 1 "74LS01N" H 5900 4600 59  0001 L BNN
 F 2 "Package_DIP:DIP-14_W7.62mm_Socket_LongPads" H 5800 4800 50  0001 C CNN
@@
 AR Path="/5E53B952/6104F018" Ref="IC?"  Part="2"
 AR Path="/60FBFA5C/6104F018" Ref="IC?"  Part="2"
-F 0 "IC?" H 5900 5425 59  0000 L BNN
+AR Path="/61043B8D/6104F018" Ref="IC9"  Part="2"
+F 0 "IC9" H 5900 5425 59  0000 L BNN
 F 1 "74LS01N" H 5900 5100 59  0001 L BNN
 F 2 "Package_DIP:DIP-14_W7.62mm_Socket_LongPads" H 5800 5300 50  0001 C CNN
@@
 AR Path="/5E53B952/6104F01E" Ref="IC?"  Part="3"
 AR Path="/60FBFA5C/6104F01E" Ref="IC?"  Part="3"
-F 0 "IC?" H 6700 3825 59  0000 L BNN
+AR Path="/61043B8D/6104F01E" Ref="IC9"  Part="3"
+F 0 "IC9" H 6700 3825 59  0000 L BNN
 F 1 "74LS01N" H 6700 3500 59  0001 L BNN
 F 2 "Package_DIP:DIP-14_W7.62mm_Socket_LongPads" H 6600 3700 50  0001 C CNN
@@
 AR Path="/5E53B952/6104F024" Ref="R?"  Part="1"
 AR Path="/60FBFA5C/6104F024" Ref="R?"  Part="1"
-F 0 "R?" V 2891 2750 59  0000 L BNN
+AR Path="/61043B8D/6104F024" Ref="R26"  Part="1"
+F 0 "R26" V 2891 2750 59  0000 L BNN
 F 1 "2K2" V 2780 2750 59  0000 L BNN
-F 2 "rosco_m68k:0207_10" H 2750 2700 50  0001 C CNN
+F 2 "rosco_m68k:R-0207_10" H 2750 2700 50  0001 C CNN
 F 3 "" H 2750 2700 50  0001 C CNN
 	1    2750 2700
@@
 AR Path="/5E53B952/6104F02A" Ref="R?"  Part="1"
 AR Path="/60FBFA5C/6104F02A" Ref="R?"  Part="1"
-F 0 "R?" H 4400 5050 59  0000 L BNN
+AR Path="/61043B8D/6104F02A" Ref="R27"  Part="1"
+F 0 "R27" H 4400 5050 59  0000 L BNN
 F 1 "270R" H 4350 5300 59  0000 L BNN
-F 2 "rosco_m68k:0207_10" H 4450 5200 50  0001 C CNN
+F 2 "rosco_m68k:R-0207_10" H 4450 5200 50  0001 C CNN
 F 3 "" H 4450 5200 50  0001 C CNN
 	1    4450 5200
@@
 AR Path="/5E53B952/6104F030" Ref="R?"  Part="1"
 AR Path="/60FBFA5C/6104F030" Ref="R?"  Part="1"
-F 0 "R?" V 8191 2850 59  0000 L BNN
+AR Path="/61043B8D/6104F030" Ref="R29"  Part="1"
+F 0 "R29" V 8191 2850 59  0000 L BNN
 F 1 "330R" V 8080 2850 59  0000 L BNN
-F 2 "rosco_m68k:0207_10" H 8050 2800 50  0001 C CNN
+F 2 "rosco_m68k:R-0207_10" H 8050 2800 50  0001 C CNN
 F 3 "" H 8050 2800 50  0001 C CNN
 	1    8050 2800
@@
 AR Path="/5E53B952/6104F036" Ref="R?"  Part="1"
 AR Path="/60FBFA5C/6104F036" Ref="R?"  Part="1"
-F 0 "R?" V 8641 2850 59  0000 L BNN
+AR Path="/61043B8D/6104F036" Ref="R30"  Part="1"
+F 0 "R30" V 8641 2850 59  0000 L BNN
 F 1 "4K7" V 8530 2850 59  0000 L BNN
-F 2 "rosco_m68k:0207_10" H 8500 2800 50  0001 C CNN
+F 2 "rosco_m68k:R-0207_10" H 8500 2800 50  0001 C CNN
 F 3 "" H 8500 2800 50  0001 C CNN
 	1    8500 2800
@@
 AR Path="/5E53B952/6104F03C" Ref="R?"  Part="1"
 AR Path="/60FBFA5C/6104F03C" Ref="R?"  Part="1"
-F 0 "R?" V 9291 2850 59  0000 L BNN
+AR Path="/61043B8D/6104F03C" Ref="R31"  Part="1"
+F 0 "R31" V 9291 2850 59  0000 L BNN
 F 1 "4K7" V 9180 2850 59  0000 L BNN
-F 2 "rosco_m68k:0207_10" H 9150 2800 50  0001 C CNN
+F 2 "rosco_m68k:R-0207_10" H 9150 2800 50  0001 C CNN
 F 3 "" H 9150 2800 50  0001 C CNN
 	1    9150 2800
@@
 AR Path="/5E53B952/6104F042" Ref="R?"  Part="1"
 AR Path="/60FBFA5C/6104F042" Ref="R?"  Part="1"
-F 0 "R?" V 7591 2850 59  0000 L BNN
+AR Path="/61043B8D/6104F042" Ref="R28"  Part="1"
+F 0 "R28" V 7591 2850 59  0000 L BNN
 F 1 "330R" V 7480 2850 59  0000 L BNN
-F 2 "rosco_m68k:0207_10" H 7450 2800 50  0001 C CNN
+F 2 "rosco_m68k:R-0207_10" H 7450 2800 50  0001 C CNN
 F 3 "" H 7450 2800 50  0001 C CNN
 	1    7450 2800
@@
 AR Path="/5E53B952/6104F048" Ref="C?"  Part="1"
 AR Path="/60FBFA5C/6104F048" Ref="C?"  Part="1"
-F 0 "C?" H 3210 2715 59  0000 L BNN
+AR Path="/61043B8D/6104F048" Ref="C11"  Part="1"
+F 0 "C11" H 3210 2715 59  0000 L BNN
 F 1 "100nF" H 3210 2515 59  0000 L BNN
 F 2 "rosco_m68k:C2.5-3" H 3150 2700 50  0001 C CNN
@@
 AR Path="/5E53B952/6104F04E" Ref="S?"  Part="1"
 AR Path="/60FBFA5C/6104F04E" Ref="S?"  Part="1"
-F 0 "S?" V 3600 5100 59  0000 L BNN
+AR Path="/61043B8D/6104F04E" Ref="S1"  Part="1"
+F 0 "S1" V 3600 5100 59  0000 L BNN
 F 1 "10-XX" V 3700 5325 59  0000 L BNN
 F 2 "rosco_m68k:B3F-10XX" H 3850 5200 50  0001 C CNN
@@
 AR Path="/5E53B952/6104F054" Ref="#SUPPLY?"  Part="1"
 AR Path="/60FBFA5C/6104F054" Ref="#SUPPLY?"  Part="1"
-F 0 "#SUPPLY?" H 2750 4700 50  0001 C CNN
+AR Path="/61043B8D/6104F054" Ref="#SUPPLY0101"  Part="1"
+F 0 "#SUPPLY0101" H 2750 4700 50  0001 C CNN
 F 1 "GND" H 2675 4575 59  0000 L BNN
 F 2 "" H 2750 4700 50  0001 C CNN
@@
 AR Path="/5E53B952/6104F05A" Ref="LED?"  Part="1"
 AR Path="/60FBFA5C/6104F05A" Ref="LED?"  Part="1"
-F 0 "LED?" H 8300 3400 59  0000 R TNN
+AR Path="/61043B8D/6104F05A" Ref="LED2"  Part="1"
+F 0 "LED2" H 8300 3400 59  0000 R TNN
 F 1 "RED" H 8300 3300 59  0000 R TNN
 F 2 "rosco_m68k:LED5MM" H 8050 3300 50  0001 C CNN
@@
 AR Path="/5E53B952/6104F060" Ref="LED?"  Part="1"
 AR Path="/60FBFA5C/6104F060" Ref="LED?"  Part="1"
-F 0 "LED?" H 7700 3400 59  0000 R TNN
+AR Path="/61043B8D/6104F060" Ref="LED1"  Part="1"
+F 0 "LED1" H 7700 3400 59  0000 R TNN
 F 1 "GREEN" H 7800 3300 59  0000 R TNN
 F 2 "rosco_m68k:LED5MM" H 7450 3300 50  0001 C CNN
@@
 AR Path="/5E53B952/6104F066" Ref="#SUPPLY?"  Part="1"
 AR Path="/60FBFA5C/6104F066" Ref="#SUPPLY?"  Part="1"
-F 0 "#SUPPLY?" H 3750 4700 50  0001 C CNN
+AR Path="/61043B8D/6104F066" Ref="#SUPPLY0102"  Part="1"
+F 0 "#SUPPLY0102" H 3750 4700 50  0001 C CNN
 F 1 "GND" H 3675 4575 59  0000 L BNN
 F 2 "" H 3750 4700 50  0001 C CNN
@@
 AR Path="/5E53B952/6104F06C" Ref="C?"  Part="1"
 AR Path="/60FBFA5C/6104F06C" Ref="C?"  Part="1"
-F 0 "C?" H 2795 4119 59  0000 L BNN
+AR Path="/61043B8D/6104F06C" Ref="C10"  Part="1"
+F 0 "C10" H 2795 4119 59  0000 L BNN
 F 1 "100uF" H 2795 3919 59  0000 L BNN
-F 2 "rosco_m68k:E2,5-5" H 2750 4100 50  0001 C CNN
+F 2 "rosco_m68k:C-Electolytic-2,5-5" H 2750 4100 50  0001 C CNN
 F 3 "" H 2750 4100 50  0001 C CNN
 	1    2750 4100
@@
 NoConn ~ 4550 3600
 $Comp
-L power:GND #PWR?
+L power:GND #PWR0126
 U 1 1 6104F076
 P 4850 5700
-F 0 "#PWR?" H 4850 5450 50  0001 C CNN
+F 0 "#PWR0126" H 4850 5450 50  0001 C CNN
 F 1 "GND" H 4855 5527 50  0000 C CNN
 F 2 "" H 4850 5700 50  0001 C CNN
@@
 	4850 5200 4850 5700
 $Comp
-L power:VCC #PWR?
+L power:VCC #PWR0127
 U 1 1 6104F07D
 P 3550 2200
-F 0 "#PWR?" H 3550 2050 50  0001 C CNN
+F 0 "#PWR0127" H 3550 2050 50  0001 C CNN
 F 1 "VCC" H 3567 2373 50  0000 C CNN
 F 2 "" H 3550 2200 50  0001 C CNN
@@
 $EndComp
 $Comp
-L power:VCC #PWR?
+L power:VCC #PWR0128
 U 1 1 6104F083
 P 4650 2200
-F 0 "#PWR?" H 4650 2050 50  0001 C CNN
+F 0 "#PWR0128" H 4650 2050 50  0001 C CNN
 F 1 "VCC" H 4667 2373 50  0000 C CNN
 F 2 "" H 4650 2200 50  0001 C CNN
@@
 $EndComp
 $Comp
-L power:VCC #PWR?
+L power:VCC #PWR0129
 U 1 1 6104F089
 P 8500 2200
-F 0 "#PWR?" H 8500 2050 50  0001 C CNN
+F 0 "#PWR0129" H 8500 2050 50  0001 C CNN
 F 1 "VCC" H 8517 2373 50  0000 C CNN
 F 2 "" H 8500 2200 50  0001 C CNN
@@
 	3550 2200 3550 3600
 $Comp
-L power:VCC #PWR?
+L power:VCC #PWR0130
 U 1 1 6104F0A4
 P 3150 2200
-F 0 "#PWR?" H 3150 2050 50  0001 C CNN
+F 0 "#PWR0130" H 3150 2050 50  0001 C CNN
 F 1 "VCC" H 3167 2373 50  0000 C CNN
 F 2 "" H 3150 2200 50  0001 C CNN
@@
 $EndComp
 $Comp
-L power:VCC #PWR?
+L power:VCC #PWR0131
 U 1 1 6104F0AA
 P 2750 2200
-F 0 "#PWR?" H 2750 2050 50  0001 C CNN
+F 0 "#PWR0131" H 2750 2050 50  0001 C CNN
 F 1 "VCC" H 2767 2373 50  0000 C CNN
 F 2 "" H 2750 2200 50  0001 C CNN

Commit message: Interrupts + Xosera schematic, re-annotate
Parts:
- renumbered C10 to C19, C11 to C20, IC10 to IC14, R26 to R29, R27 to R30, R28 to R31, R29 to R32, R30 to R33, R31 to R34
Changed lines of the file:
@@
 $Descr A4 11693 8268
 encoding utf-8
-Sheet 8 10
+Sheet 8 13
 Title "rosco_m68k Pro (030) Prototype"
 Date "2021-07-24"
@@
 AR Path="/5E53B952/6104F00C" Ref="IC?"  Part="1"
 AR Path="/60FBFA5C/6104F00C" Ref="IC?"  Part="1"
-AR Path="/61043B8D/6104F00C" Ref="IC10"  Part="1"
-F 0 "IC10" H 3850 4130 59  0000 L BNN
+AR Path="/61043B8D/6104F00C" Ref="IC14"  Part="1"
+F 0 "IC14" H 3850 4130 59  0000 L BNN
 F 1 "555N" H 3850 3195 59  0000 L BNN
 F 2 "Package_DIP:DIP-8_W7.62mm_LongPads" H 4150 3700 50  0001 C CNN
@@
 AR Path="/5E53B952/6104F024" Ref="R?"  Part="1"
 AR Path="/60FBFA5C/6104F024" Ref="R?"  Part="1"
-AR Path="/61043B8D/6104F024" Ref="R26"  Part="1"
-F 0 "R26" V 2891 2750 59  0000 L BNN
+AR Path="/61043B8D/6104F024" Ref="R29"  Part="1"
+F 0 "R29" V 2891 2750 59  0000 L BNN
 F 1 "2K2" V 2780 2750 59  0000 L BNN
 F 2 "rosco_m68k:R-0207_10" H 2750 2700 50  0001 C CNN
@@
 AR Path="/5E53B952/6104F02A" Ref="R?"  Part="1"
 AR Path="/60FBFA5C/6104F02A" Ref="R?"  Part="1"
-AR Path="/61043B8D/6104F02A" Ref="R27"  Part="1"
-F 0 "R27" H 4400 5050 59  0000 L BNN
+AR Path="/61043B8D/6104F02A" Ref="R30"  Part="1"
+F 0 "R30" H 4400 5050 59  0000 L BNN
 F 1 "270R" H 4350 5300 59  0000 L BNN
 F 2 "rosco_m68k:R-0207_10" H 4450 5200 50  0001 C CNN
@@
 AR Path="/5E53B952/6104F030" Ref="R?"  Part="1"
 AR Path="/60FBFA5C/6104F030" Ref="R?"  Part="1"
-AR Path="/61043B8D/6104F030" Ref="R29"  Part="1"
-F 0 "R29" V 8191 2850 59  0000 L BNN
+AR Path="/61043B8D/6104F030" Ref="R32"  Part="1"
+F 0 "R32" V 8191 2850 59  0000 L BNN
 F 1 "330R" V 8080 2850 59  0000 L BNN
 F 2 "rosco_m68k:R-0207_10" H 8050 2800 50  0001 C CNN
@@
 AR Path="/5E53B952/6104F036" Ref="R?"  Part="1"
 AR Path="/60FBFA5C/6104F036" Ref="R?"  Part="1"
-AR Path="/61043B8D/6104F036" Ref="R30"  Part="1"
-F 0 "R30" V 8641 2850 59  0000 L BNN
+AR Path="/61043B8D/6104F036" Ref="R33"  Part="1"
+F 0 "R33" V 8641 2850 59  0000 L BNN
 F 1 "4K7" V 8530 2850 59  0000 L BNN
 F 2 "rosco_m68k:R-0207_10" H 8500 2800 50  0001 C CNN
@@
 AR Path="/5E53B952/6104F03C" Ref="R?"  Part="1"
 AR Path="/60FBFA5C/6104F03C" Ref="R?"  Part="1"
-AR Path="/61043B8D/6104F03C" Ref="R31"  Part="1"
-F 0 "R31" V 9291 2850 59  0000 L BNN
+AR Path="/61043B8D/6104F03C" Ref="R34"  Part="1"
+F 0 "R34" V 9291 2850 59  0000 L BNN
 F 1 "4K7" V 9180 2850 59  0000 L BNN
 F 2 "rosco_m68k:R-0207_10" H 9150 2800 50  0001 C CNN
@@
 AR Path="/5E53B952/6104F042" Ref="R?"  Part="1"
 AR Path="/60FBFA5C/6104F042" Ref="R?"  Part="1"
-AR Path="/61043B8D/6104F042" Ref="R28"  Part="1"
-F 0 "R28" V 7591 2850 59  0000 L BNN
+AR Path="/61043B8D/6104F042" Ref="R31"  Part="1"
+F 0 "R31" V 7591 2850 59  0000 L BNN
 F 1 "330R" V 7480 2850 59  0000 L BNN
 F 2 "rosco_m68k:R-0207_10" H 7450 2800 50  0001 C CNN
@@
 AR Path="/5E53B952/6104F048" Ref="C?"  Part="1"
 AR Path="/60FBFA5C/6104F048" Ref="C?"  Part="1"
-AR Path="/61043B8D/6104F048" Ref="C11"  Part="1"
-F 0 "C11" H 3210 2715 59  0000 L BNN
+AR Path="/61043B8D/6104F048" Ref="C20"  Part="1"
+F 0 "C20" H 3210 2715 59  0000 L BNN
 F 1 "100nF" H 3210 2515 59  0000 L BNN
 F 2 "rosco_m68k:C2.5-3" H 3150 2700 50  0001 C CNN
@@
 AR Path="/5E53B952/6104F054" Ref="#SUPPLY?"  Part="1"
 AR Path="/60FBFA5C/6104F054" Ref="#SUPPLY?"  Part="1"
-AR Path="/61043B8D/6104F054" Ref="#SUPPLY0101"  Part="1"
-F 0 "#SUPPLY0101" H 2750 4700 50  0001 C CNN
+AR Path="/61043B8D/6104F054" Ref="#SUPPLY01"  Part="1"
+F 0 "#SUPPLY01" H 2750 4700 50  0001 C CNN
 F 1 "GND" H 2675 4575 59  0000 L BNN
 F 2 "" H 2750 4700 50  0001 C CNN
@@
 AR Path="/5E53B952/6104F066" Ref="#SUPPLY?"  Part="1"
 AR Path="/60FBFA5C/6104F066" Ref="#SUPPLY?"  Part="1"
-AR Path="/61043B8D/6104F066" Ref="#SUPPLY0102"  Part="1"
-F 0 "#SUPPLY0102" H 3750 4700 50  0001 C CNN
+AR Path="/61043B8D/6104F066" Ref="#SUPPLY02"  Part="1"
+F 0 "#SUPPLY02" H 3750 4700 50  0001 C CNN
 F 1 "GND" H 3675 4575 59  0000 L BNN
 F 2 "" H 3750 4700 50  0001 C CNN
@@
 AR Path="/5E53B952/6104F06C" Ref="C?"  Part="1"
 AR Path="/60FBFA5C/6104F06C" Ref="C?"  Part="1"
-AR Path="/61043B8D/6104F06C" Ref="C10"  Part="1"
-F 0 "C10" H 2795 4119 59  0000 L BNN
+AR Path="/61043B8D/6104F06C" Ref="C19"  Part="1"
+F 0 "C19" H 2795 4119 59  0000 L BNN
 F 1 "100uF" H 2795 3919 59  0000 L BNN
 F 2 "rosco_m68k:C-Electolytic-2,5-5" H 2750 4100 50  0001 C CNN
@@
 NoConn ~ 4550 3600
 $Comp
-L power:GND #PWR0126
+L power:GND #PWR037
 U 1 1 6104F076
 P 4850 5700
-F 0 "#PWR0126" H 4850 5450 50  0001 C CNN
+F 0 "#PWR037" H 4850 5450 50  0001 C CNN
 F 1 "GND" H 4855 5527 50  0000 C CNN
 F 2 "" H 4850 5700 50  0001 C CNN
@@
 	4850 5200 4850 5700
 $Comp
-L power:VCC #PWR0127
+L power:VCC #PWR035
 U 1 1 6104F07D
 P 3550 2200
-F 0 "#PWR0127" H 3550 2050 50  0001 C CNN
+F 0 "#PWR035" H 3550 2050 50  0001 C CNN
 F 1 "VCC" H 3567 2373 50  0000 C CNN
 F 2 "" H 3550 2200 50  0001 C CNN
@@
 $EndComp
 $Comp
-L power:VCC #PWR0128
+L power:VCC #PWR036
 U 1 1 6104F083
 P 4650 2200
-F 0 "#PWR0128" H 4650 2050 50  0001 C CNN
+F 0 "#PWR036" H 4650 2050 50  0001 C CNN
 F 1 "VCC" H 4667 2373 50  0000 C CNN
 F 2 "" H 4650 2200 50  0001 C CNN
@@
 $EndComp
 $Comp
-L power:VCC #PWR0129
+L power:VCC #PWR038
 U 1 1 6104F089
 P 8500 2200
-F 0 "#PWR0129" H 8500 2050 50  0001 C CNN
+F 0 "#PWR038" H 8500 2050 50  0001 C CNN
 F 1 "VCC" H 8517 2373 50  0000 C CNN
 F 2 "" H 8500 2200 50  0001 C CNN
@@
 	3550 2200 3550 3600
 $Comp
-L power:VCC #PWR0130
+L power:VCC #PWR034
 U 1 1 6104F0A4
 P 3150 2200
-F 0 "#PWR0130" H 3150 2050 50  0001 C CNN
+F 0 "#PWR034" H 3150 2050 50  0001 C CNN
 F 1 "VCC" H 3167 2373 50  0000 C CNN
 F 2 "" H 3150 2200 50  0001 C CNN
@@
 $EndComp
 $Comp
-L power:VCC #PWR0131
+L power:VCC #PWR033
 U 1 1 6104F0AA
 P 2750 2200
-F 0 "#PWR0131" H 2750 2050 50  0001 C CNN
+F 0 "#PWR033" H 2750 2050 50  0001 C CNN
 F 1 "VCC" H 2767 2373 50  0000 C CNN
 F 2 "" H 2750 2200 50  0001 C CNN

Commit message: Big(ish) push on placement
Parts:
- C20: footprint rosco_m68k:C2.5-3 -> Capacitor_THT:C_Rect_L4.0mm_W2.5mm_P2.50mm
Changed lines of the file:
@@
 F 0 "C20" H 3210 2715 59  0000 L BNN
 F 1 "100nF" H 3210 2515 59  0000 L BNN
-F 2 "rosco_m68k:C2.5-3" H 3150 2700 50  0001 C CNN
+F 2 "Capacitor_THT:C_Rect_L4.0mm_W2.5mm_P2.50mm" H 3150 2700 50  0001 C CNN
 F 3 "" H 3150 2700 50  0001 C CNN
 	1    3150 2700

Commit message: Further layout
Parts:
- renumbered C19 to C18, C20 to C19, IC14 to IC13, IC9 to IC8, R29 to R27, R30 to R28, R31 to R29, R32 to R30, R33 to R31, R34 to R32
Changed lines of the file:
@@
 AR Path="/5E53B952/6104F00C" Ref="IC?"  Part="1"
 AR Path="/60FBFA5C/6104F00C" Ref="IC?"  Part="1"
-AR Path="/61043B8D/6104F00C" Ref="IC14"  Part="1"
-F 0 "IC14" H 3850 4130 59  0000 L BNN
+AR Path="/61043B8D/6104F00C" Ref="IC13"  Part="1"
+F 0 "IC13" H 3850 4130 59  0000 L BNN
 F 1 "555N" H 3850 3195 59  0000 L BNN
 F 2 "Package_DIP:DIP-8_W7.62mm_LongPads" H 4150 3700 50  0001 C CNN
@@
 AR Path="/5E53B952/6104F012" Ref="IC?"  Part="1"
 AR Path="/60FBFA5C/6104F012" Ref="IC?"  Part="1"
-AR Path="/61043B8D/6104F012" Ref="IC9"  Part="1"
-F 0 "IC9" H 5900 4925 59  0000 L BNN
+AR Path="/61043B8D/6104F012" Ref="IC8"  Part="1"
+F 0 "IC8" H 5900 4925 59  0000 L BNN
 F 1 "74LS01N" H 5900 4600 59  0001 L BNN
 F 2 "Package_DIP:DIP-14_W7.62mm_Socket_LongPads" H 5800 4800 50  0001 C CNN
@@
 AR Path="/5E53B952/6104F018" Ref="IC?"  Part="2"
 AR Path="/60FBFA5C/6104F018" Ref="IC?"  Part="2"
-AR Path="/61043B8D/6104F018" Ref="IC9"  Part="2"
-F 0 "IC9" H 5900 5425 59  0000 L BNN
+AR Path="/61043B8D/6104F018" Ref="IC8"  Part="2"
+F 0 "IC8" H 5900 5425 59  0000 L BNN
 F 1 "74LS01N" H 5900 5100 59  0001 L BNN
 F 2 "Package_DIP:DIP-14_W7.62mm_Socket_LongPads" H 5800 5300 50  0001 C CNN
@@
 AR Path="/5E53B952/6104F01E" Ref="IC?"  Part="3"
 AR Path="/60FBFA5C/6104F01E" Ref="IC?"  Part="3"
-AR Path="/61043B8D/6104F01E" Ref="IC9"  Part="3"
-F 0 "IC9" H 6700 3825 59  0000 L BNN
+AR Path="/61043B8D/6104F01E" Ref="IC8"  Part="3"
+F 0 "IC8" H 6700 3825 59  0000 L BNN
 F 1 "74LS01N" H 6700 3500 59  0001 L BNN
 F 2 "Package_DIP:DIP-14_W7.62mm_Socket_LongPads" H 6600 3700 50  0001 C CNN
@@
 AR Path="/5E53B952/6104F024" Ref="R?"  Part="1"
 AR Path="/60FBFA5C/6104F024" Ref="R?"  Part="1"
-AR Path="/61043B8D/6104F024" Ref="R29"  Part="1"
-F 0 "R29" V 2891 2750 59  0000 L BNN
+AR Path="/61043B8D/6104F024" Ref="R27"  Part="1"
+F 0 "R27" V 2891 2750 59  0000 L BNN
 F 1 "2K2" V 2780 2750 59  0000 L BNN
 F 2 "rosco_m68k:R-0207_10" H 2750 2700 50  0001 C CNN
@@
 AR Path="/5E53B952/6104F02A" Ref="R?"  Part="1"
 AR Path="/60FBFA5C/6104F02A" Ref="R?"  Part="1"
-AR Path="/61043B8D/6104F02A" Ref="R30"  Part="1"
-F 0 "R30" H 4400 5050 59  0000 L BNN
+AR Path="/61043B8D/6104F02A" Ref="R28"  Part="1"
+F 0 "R28" H 4400 5050 59  0000 L BNN
 F 1 "270R" H 4350 5300 59  0000 L BNN
 F 2 "rosco_m68k:R-0207_10" H 4450 5200 50  0001 C CNN
@@
 AR Path="/5E53B952/6104F030" Ref="R?"  Part="1"
 AR Path="/60FBFA5C/6104F030" Ref="R?"  Part="1"
-AR Path="/61043B8D/6104F030" Ref="R32"  Part="1"
-F 0 "R32" V 8191 2850 59  0000 L BNN
+AR Path="/61043B8D/6104F030" Ref="R30"  Part="1"
+F 0 "R30" V 8191 2850 59  0000 L BNN
 F 1 "330R" V 8080 2850 59  0000 L BNN
 F 2 "rosco_m68k:R-0207_10" H 8050 2800 50  0001 C CNN
@@
 AR Path="/5E53B952/6104F036" Ref="R?"  Part="1"
 AR Path="/60FBFA5C/6104F036" Ref="R?"  Part="1"
-AR Path="/61043B8D/6104F036" Ref="R33"  Part="1"
-F 0 "R33" V 8641 2850 59  0000 L BNN
+AR Path="/61043B8D/6104F036" Ref="R31"  Part="1"
+F 0 "R31" V 8641 2850 59  0000 L BNN
 F 1 "4K7" V 8530 2850 59  0000 L BNN
 F 2 "rosco_m68k:R-0207_10" H 8500 2800 50  0001 C CNN
@@
 AR Path="/5E53B952/6104F03C" Ref="R?"  Part="1"
 AR Path="/60FBFA5C/6104F03C" Ref="R?"  Part="1"
-AR Path="/61043B8D/6104F03C" Ref="R34"  Part="1"
-F 0 "R34" V 9291 2850 59  0000 L BNN
+AR Path="/61043B8D/6104F03C" Ref="R32"  Part="1"
+F 0 "R32" V 9291 2850 59  0000 L BNN
 F 1 "4K7" V 9180 2850 59  0000 L BNN
 F 2 "rosco_m68k:R-0207_10" H 9150 2800 50  0001 C CNN
@@
 AR Path="/5E53B952/6104F042" Ref="R?"  Part="1"
 AR Path="/60FBFA5C/6104F042" Ref="R?"  Part="1"
-AR Path="/61043B8D/6104F042" Ref="R31"  Part="1"
-F 0 "R31" V 7591 2850 59  0000 L BNN
+AR Path="/61043B8D/6104F042" Ref="R29"  Part="1"
+F 0 "R29" V 7591 2850 59  0000 L BNN
 F 1 "330R" V 7480 2850 59  0000 L BNN
 F 2 "rosco_m68k:R-0207_10" H 7450 2800 50  0001 C CNN
@@
 AR Path="/5E53B952/6104F048" Ref="C?"  Part="1"
 AR Path="/60FBFA5C/6104F048" Ref="C?"  Part="1"
-AR Path="/61043B8D/6104F048" Ref="C20"  Part="1"
-F 0 "C20" H 3210 2715 59  0000 L BNN
+AR Path="/61043B8D/6104F048" Ref="C19"  Part="1"
+F 0 "C19" H 3210 2715 59  0000 L BNN
 F 1 "100nF" H 3210 2515 59  0000 L BNN
 F 2 "Capacitor_THT:C_Rect_L4.0mm_W2.5mm_P2.50mm" H 3150 2700 50  0001 C CNN
@@
 AR Path="/5E53B952/6104F06C" Ref="C?"  Part="1"
 AR Path="/60FBFA5C/6104F06C" Ref="C?"  Part="1"
-AR Path="/61043B8D/6104F06C" Ref="C19"  Part="1"
-F 0 "C19" H 2795 4119 59  0000 L BNN
+AR Path="/61043B8D/6104F06C" Ref="C18"  Part="1"
+F 0 "C18" H 2795 4119 59  0000 L BNN
 F 1 "100uF" H 2795 3919 59  0000 L BNN
 F 2 "rosco_m68k:C-Electolytic-2,5-5" H 2750 4100 50  0001 C CNN
@@
 NoConn ~ 4550 3600
 $Comp
-L power:GND #PWR037
+L power:GND #PWR036
 U 1 1 6104F076
 P 4850 5700
-F 0 "#PWR037" H 4850 5450 50  0001 C CNN
+F 0 "#PWR036" H 4850 5450 50  0001 C CNN
 F 1 "GND" H 4855 5527 50  0000 C CNN
 F 2 "" H 4850 5700 50  0001 C CNN
@@
 	4850 5200 4850 5700
 $Comp
-L power:VCC #PWR035
+L power:VCC #PWR034
 U 1 1 6104F07D
 P 3550 2200
-F 0 "#PWR035" H 3550 2050 50  0001 C CNN
+F 0 "#PWR034" H 3550 2050 50  0001 C CNN
 F 1 "VCC" H 3567 2373 50  0000 C CNN
 F 2 "" H 3550 2200 50  0001 C CNN
@@
 $EndComp
 $Comp
-L power:VCC #PWR036
+L power:VCC #PWR035
 U 1 1 6104F083
 P 4650 2200
-F 0 "#PWR036" H 4650 2050 50  0001 C CNN
+F 0 "#PWR035" H 4650 2050 50  0001 C CNN
 F 1 "VCC" H 4667 2373 50  0000 C CNN
 F 2 "" H 4650 2200 50  0001 C CNN
@@
 $EndComp
 $Comp
-L power:VCC #PWR038
+L power:VCC #PWR037
 U 1 1 6104F089
 P 8500 2200
-F 0 "#PWR038" H 8500 2050 50  0001 C CNN
+F 0 "#PWR037" H 8500 2050 50  0001 C CNN
 F 1 "VCC" H 8517 2373 50  0000 C CNN
 F 2 "" H 8500 2200 50  0001 C CNN
@@
 	3550 2200 3550 3600
 $Comp
-L power:VCC #PWR034
+L power:VCC #PWR033
 U 1 1 6104F0A4
 P 3150 2200
-F 0 "#PWR034" H 3150 2050 50  0001 C CNN
+F 0 "#PWR033" H 3150 2050 50  0001 C CNN
 F 1 "VCC" H 3167 2373 50  0000 C CNN
 F 2 "" H 3150 2200 50  0001 C CNN
@@
 $EndComp
 $Comp
-L power:VCC #PWR033
+L power:VCC #PWR032
 U 1 1 6104F0AA
 P 2750 2200
-F 0 "#PWR033" H 2750 2050 50  0001 C CNN
+F 0 "#PWR032" H 2750 2050 50  0001 C CNN
 F 1 "VCC" H 2767 2373 50  0000 C CNN
 F 2 "" H 2750 2200 50  0001 C CNN
