File: design/pro_030_proto/kicad/UNUSED.sch (KiCad schematic (older format))
At the start: 10 parts, among them IC14 74LS05

Commit message: Replace 7493s and 7404 with IC10 GAL
Parts:
- added unit 4 of IC14
Connections:
- no-connect marks 1 -> 2
Changed lines of the file:
@@
 GND
 NoConn ~ 5250 3850
+$Comp
+L 74xx:74LS05 IC14
+U 4 1 615F8F5E
+P 4950 3300
+F 0 "IC14" H 4950 3617 50  0000 C CNN
+F 1 "74LS05" H 4950 3526 50  0000 C CNN
+F 2 "" H 4950 3300 50  0001 C CNN
+F 3 "http://www.ti.com/lit/gpn/sn74LS05" H 4950 3300 50  0001 C CNN
+	4    4950 3300
+	1    0    0    -1
+$EndComp
+Text GLabel 4650 3300 0    50   UnSpc ~ 0
+GND
+NoConn ~ 5250 3300
 $EndSCHEMATC

Commit message: Add IC14 GAL into schematic
Parts:
- removed IC14: 74LS05, symbol 74xx:74LS05
Connections:
- no-connect marks 2 -> 0
Changed lines of the file:
@@
 	3800 1750 3800 1900
 Connection ~ 3800 1900
-$Comp
-L 74xx:74LS05 IC14
-U 6 1 61721131
-P 4950 3850
-F 0 "IC14" H 4950 4167 50  0000 C CNN
-F 1 "74LS05" H 4950 4076 50  0000 C CNN
-F 2 "" H 4950 3850 50  0001 C CNN
-F 3 "http://www.ti.com/lit/gpn/sn74LS05" H 4950 3850 50  0001 C CNN
-	6    4950 3850
-	1    0    0    -1
-$EndComp
-Text GLabel 4650 3850 0    50   UnSpc ~ 0
-GND
-NoConn ~ 5250 3850
-$Comp
-L 74xx:74LS05 IC14
-U 4 1 615F8F5E
-P 4950 3300
-F 0 "IC14" H 4950 3617 50  0000 C CNN
-F 1 "74LS05" H 4950 3526 50  0000 C CNN
-F 2 "" H 4950 3300 50  0001 C CNN
-F 3 "http://www.ti.com/lit/gpn/sn74LS05" H 4950 3300 50  0001 C CNN
-	4    4950 3300
-	1    0    0    -1
-$EndComp
-Text GLabel 4650 3300 0    50   UnSpc ~ 0
-GND
-NoConn ~ 5250 3300
 $EndSCHEMATC
