File: design/pro_030_proto/kicad/INTERFACE.sch (KiCad schematic (older format))
At the start: 7 parts, among them IC30 PCF8584, J17 DIN41612_96, J19 DIN41612_96, J22 DIN41612_96, J24 I2C, J25 Conn_01x06_Male

Commit message: More tidy up & swap layers
Connections:
- net SDA: now reaches IC30.2 (SDA), J24.2 (Pin_2)
- net SCL: now reaches IC30.3 (SCL), J24.1 (Pin_1)
Changed lines of the file:
@@
 Text GLabel 2450 6650 2    50   UnSpc ~ 0
 GND
+Text Label 3600 3350 2    50   ~ 0
+SDA
+Text Label 3600 3550 2    50   ~ 0
+SCL
 $EndSCHEMATC
